Commit message: modified:   franka_description/robots/common/franka_arm.xacro modified:   franka_example_controllers/scripts/interactive_marker.py modified:   franka_example_controllers/scripts/move_to_start.py

File: franka_description/robots/common/franka_arm.xacro (robot description, xacro)
@@ -113,5 +113,5 @@
     <link name="${arm_id}_link8"/>
     <joint name="${arm_id}_joint8" type="fixed">
-      <origin rpy="0 0 0" xyz="0 0 0.107"/>
+      <origin rpy=" 0 0 ${-pi/4}" xyz="0 0 0.107"/>
       <parent link="${arm_id}_link7"/>
       <child link="${arm_id}_link8"/>
